Commit message: Update hitbot urdf files

File: handson_description/urdf/hitbot/hitbot.gazebo.xacro (robot description, xacro)
@@ -1,8 +1,23 @@
 <?xml version='1.0' encoding='utf-8'?>
 <robot xmlns:xacro="http://www.ros.org/wiki/xacro" name="hitbot_gazebo">
-	<gazebo reference="hitbot_base"><material>Gazebo/Black</material></gazebo>
-	<gazebo reference="hitbot_mask"></gazebo>
-	<gazebo reference="hitbot_finger0"><material>Gazebo/Grey</material></gazebo>
-	<gazebo reference="hitbot_finger1"><material>Gazebo/Grey</material></gazebo>
+	<gazebo reference="hitbot_base">
+    <material>Gazebo/Black</material>
+    <mu1>0.9</mu1>
+    <mu2>0.9</mu2>
+  </gazebo>
+	<gazebo reference="hitbot_mask">
+    <mu1>0.9</mu1>
+    <mu2>0.9</mu2>
+  </gazebo>
+	<gazebo reference="hitbot_finger0">
+    <material>Gazebo/Grey</material>
+    <mu1>0.9</mu1>
+    <mu2>0.9</mu2>
+  </gazebo>
+	<gazebo reference="hitbot_finger1">
+    <material>Gazebo/Grey</material>
+    <mu1>0.9</mu1>
+    <mu2>0.9</mu2>
+  </gazebo>
 	<transmission name="hitbot_finger_joint1_trans">
     <type>transmission_interface/SimpleTransmission</type>
@@ -12,4 +27,5 @@
     <actuator name="hitbot_finger_joint1_motor">
       <mechanicalReduction>1</mechanicalReduction>
+      <hardwareInterface>hardware_interface/PositionJointInterface</hardwareInterface>
     </actuator>
   </transmission>
@@ -21,4 +37,5 @@
     <actuator name="hitbot_finger_joint2_motor">
       <mechanicalReduction>1</mechanicalReduction>
+      <hardwareInterface>hardware_interface/PositionJointInterface</hardwareInterface>
     </actuator>
   </transmission>

File: handson_description/urdf/hitbot/hitbot.urdf.xacro (robot description, xacro)
@@ -9,7 +9,7 @@
   <link name="hitbot_base">
     <inertial>
-      <mass value="0.73" />
+      <mass value="0.1" />
       <origin xyz="0 0.0015244 0.0275912" rpy="0 0 0" />
-      <inertia ixx="0.00278560230025" ixy="0.0" ixz="0.0" iyy="0.000400033405336" iyz="0.0" izz="0.00256378041832" />
+      <inertia ixx="3.01220925051e-05" ixy="0.0" ixz="0.0" iyy="2.95873808038e-05" iyz="0.0" izz="6.95125211657e-06" />
     </inertial>
     <visual>
@@ -32,5 +32,5 @@
       <mass value="0.1" />
       <origin xyz="0 0.0015244 0.0275912" rpy="0 0 0" />
-      <inertia ixx="0.003" ixy="0.0" ixz="0.0" iyy="0.003" iyz="0.0" izz="0.003" />
+      <inertia ixx="3.01220925051e-05" ixy="0.0" ixz="0.0" iyy="2.95873808038e-05" iyz="0.0" izz="6.95125211657e-06" />
     </inertial>
     <visual>
@@ -79,5 +79,5 @@
     <child link="hitbot_finger0"/>
     <axis xyz="0 1 0"/>
-    <limit upper="0" lower="-0.010" effort="30" velocity="0.01"/>
+    <limit upper="0" lower="-0.010" effort="1000" velocity="0.01"/>
   </joint>
   <!-- finger 0 tip -->
@@ -133,5 +133,5 @@
     <child link="hitbot_finger1"/>
     <axis xyz="0 1 0"/>
-    <limit upper="0.010" lower="0" effort="30" velocity="0.01"/>
+    <limit upper="0.010" lower="0" effort="1000" velocity="0.01"/>
   </joint>
   <!-- finger 0 tip -->
